Commit message: updated sensor xacro

File: my_sensor_kit_description/urdf/sensor_kit.xacro (robot description, xacro)
@@ -20,12 +20,18 @@
     <xacro:property name="calibration" value="${xacro.load_yaml('$(arg config_dir)/sensor_kit_calibration.yaml')}"/>
     <!-- lidar -->
-    <xacro:VLP-16 parent="sensor_kit_base_link" name="velodyne" topic="/velodyne_points" hz="10" samples="220" gpu="$(arg gpu)">
+    <xacro:VLP-16
+	parent="sensor_kit_base_link"
+	name="velodyne_top"
+	topic="/points_raw"
+	hz="10"
+	samples="220"
+	gpu="$(arg gpu)">
       <origin
-        xyz="${calibration['sensor_kit_base_link']['velodyne_base_link']['x']}
-             ${calibration['sensor_kit_base_link']['velodyne_base_link']['y']}
-             ${calibration['sensor_kit_base_link']['velodyne_base_link']['z']}"
-        rpy="${calibration['sensor_kit_base_link']['velodyne_base_link']['roll']}
-             ${calibration['sensor_kit_base_link']['velodyne_base_link']['pitch']}
-             ${calibration['sensor_kit_base_link']['velodyne_base_link']['yaw']}"
+        xyz="${calibration['sensor_kit_base_link']['velodyne_top_base_link']['x']}
+             ${calibration['sensor_kit_base_link']['velodyne_top_base_link']['y']}
+             ${calibration['sensor_kit_base_link']['velodyne_top_base_link']['z']}"
+        rpy="${calibration['sensor_kit_base_link']['velodyne_top_base_link']['roll']}
+             ${calibration['sensor_kit_base_link']['velodyne_top_base_link']['pitch']}
+             ${calibration['sensor_kit_base_link']['velodyne_top_base_link']['yaw']}"
       />
     </xacro:VLP-16>

File: my_sensor_kit_description/urdf/sensors.xacro (robot description, xacro)
@@ -15,14 +15,3 @@
   />
   <!-- embedded sensors -->
-  <xacro:include filename="$(find velodyne_description)/urdf/VLP-16.urdf.xacro"/>
-  <xacro:VLP-16 parent="base_link" name="velodyne_rear" topic="/velodyne_points" hz="10" samples="220" gpu="false">
-    <origin
-      xyz="${calibration['base_link']['velodyne_base_link']['x']}
-           ${calibration['base_link']['velodyne_base_link']['y']}
-           ${calibration['base_link']['velodyne_base_link']['z']}"
-      rpy="${calibration['base_link']['velodyne_base_link']['roll']}
-           ${calibration['base_link']['velodyne_base_link']['pitch']}
-           ${calibration['base_link']['velodyne_base_link']['yaw']}"
-    />
-  </xacro:VLP-16>
 </robot>
